File: schematics/WindStation.brd (EAGLE design)
At the start: 35.2 x 39.4 mm, 8 parts

Commit message: Update schematic
Parts:
- removed JP2: (no value), pinhead:1X02
- removed JP3: DHT, adafruit:1X03
- added DHT: DHT, adafruit:1X03
- added MGT2: BEAGLEBONEBLACK_MOUNTING_HOLE, BeagleBone_Black_Wireless:BEAGLEBONEBLACK_MOUNTING_HOLE
- added PWR, WIND: (no value), pinhead:1X02
- JP1: value Pyranometer -> Pyro
- moved JP1 8.26 mm to (32.0, 15.9)
Connections:
- net 0: now also DHT.3, MGT2.P$1, PWR.1, WIND.2; no longer JP2.2, JP3.3
- net N$3: now also WIND.1; no longer JP2.1
- net N$4: now also DHT.2; no longer JP3.2
- net VCC: now also DHT.1, PWR.2; no longer JP3.1
Routing:
- net VCC: track 29.9 -> 39.3 mm
- net N$3: track 31.0 -> 26.9 mm
- net N$1: track 12.3 -> 15.7 mm
- net 0: track 51.6 -> 54.6 mm
- net N$4: track 10.9 -> 9.27 mm
Other:
- board text added: "+"
- board text added: "G"
