File: schematics/WindStation.sch (EAGLE design)
At the start: 8 parts

Commit message: Update schematic
Parts:
- removed JP2: (no value), pinhead:PINHD-1X2
- removed JP3: DHT, adafruit:PINHD-1X3
- added DHT: DHT, adafruit:PINHD-1X3
- added MGT2: BEAGLEBONEBLACK_MOUNTING_HOLE, BeagleBone_Black_Wireless:BEAGLEBONEBLACK_MOUNTING_HOLE
- added PWR, WIND: (no value), pinhead:PINHD-1X2
- JP1: value Pyranometer -> Pyro
Connections:
- net 0: now also DHT.3, MGT2.P$1, PWR.1, WIND.2; no longer JP2.2, JP3.3
- net N$3: now also WIND.1; no longer JP2.1
- net N$4: now also DHT.2; no longer JP3.2
- net VCC: now also DHT.1, PWR.2; no longer JP3.1
Other:
- moved on the sheet: R3
